File: hardware/rpi-cm4-base-carrier/cm4-gpio.kicad_sch (KiCad schematic)
At the start: 15 parts, among them J1 DNP, J2 USB4105-GF-A, J3 SM04B-SRSS-TB(LF)(SN), U1 74LVC1G07SE-7

Commit message: updated metadata
Other:
- title: Raspberry Pi Compute Module 4 Base Carrier -> CM4 Carrier
