File: hardware/rpi-cm4-base-carrier/cm4-high-speed.kicad_sch (KiCad schematic)
At the start: 5 parts, among them J4 USB_OTG, U2 TPD2EUSB30

Commit message: updated metadata
Other:
- title: Raspberry Pi Compute Module 4 Base Carrier -> CM4 Carrier
