File: hardware/rpi-cm4-base-carrier/rpi-cm4-base-carrier.kicad_sch (KiCad schematic)
At the start: 0 parts

Commit message: updated metadata
Other:
- title: Raspberry Pi Compute Module 4 Base Carrier -> CM4 Base
Changed lines of the file:
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@@
-(kicad_sch (version 20201015) (generator eeschema)
-  (page 1 3)
+(kicad_sch (version 20211123) (generator eeschema)
   (paper "A4")
   (title_block
-    (title "Raspberry Pi Compute Module 4 Base Carrier")
-    (date "2020-10-31")
+    (title "CM4 Base")
+    (date "01/22/2022")
     (rev "v01")
     (comment 2 "creativecommons.org/licenses/by-sa/4.0/")
     (comment 3 "License: CC BY-SA 4.0")
-    (comment 4 "Author: Shawn Hymel")
+    (comment 4 "Author: Devin Henkel-Legare")
+  )
+  (sheet (at 101.6 101.6) (size 38.1 38.1)
+    (stroke (width 0) (type solid) (color 132 0 132 1))
+    (fill (color 255 255 255 0.0000))
+    (property "Sheet name" "CM4 High Speed" (id 0) (at 101.6 100.9645 0)
+      (effects (font (size 1.27 1.27)) (justify left bottom))
+    )
+    (property "Sheet file" "cm4-high-speed.kicad_sch" (id 1) (at 101.6 140.2085 0)
+      (effects (font (size 1.27 1.27)) (justify left top))
+    )
   )
   (sheet (at 101.6 50.8) (size 38.1 38.1)
@@
     )
   )
-  (sheet (at 101.6 101.6) (size 38.1 38.1)
-    (stroke (width 0) (type solid) (color 132 0 132 1))
-    (fill (color 255 255 255 0.0000))
-    (property "Sheet name" "CM4 High Speed" (id 0) (at 101.6 100.9645 0)
-      (effects (font (size 1.27 1.27)) (justify left bottom))
-    )
-    (property "Sheet file" "cm4-high-speed.kicad_sch" (id 1) (at 101.6 140.2085 0)
-      (effects (font (size 1.27 1.27)) (justify left top))
-    )
-  )
   (sheet_instances
     (path "/" (page "1"))
-    (path "/fc4c71a5-1008-4ac4-98db-57c838c57d91/" (page "3"))
-    (path "/caa71f4c-454d-4ac9-b287-456eafb34991/" (page "3"))
+    (path "/fc4c71a5-1008-4ac4-98db-57c838c57d91" (page "3"))
+    (path "/caa71f4c-454d-4ac9-b287-456eafb34991" (page "3"))
   )
   (symbol_instances
@@
       (reference "#PWR0110") (unit 1) (value "GND") (footprint "")
     )
+    (path "/caa71f4c-454d-4ac9-b287-456eafb34991/0d0caf91-4ece-48ed-a178-43a8b49f3526"
+      (reference "#PWR0111") (unit 1) (value "GND") (footprint "")
+    )
+    (path "/caa71f4c-454d-4ac9-b287-456eafb34991/81f0d702-912e-410d-83f3-c9f3bd3f7f28"
+      (reference "#PWR0112") (unit 1) (value "GND") (footprint "")
+    )
+    (path "/caa71f4c-454d-4ac9-b287-456eafb34991/7aaeccae-7554-4237-a159-f19729377488"
+      (reference "#PWR0113") (unit 1) (value "GND") (footprint "")
+    )
+    (path "/caa71f4c-454d-4ac9-b287-456eafb34991/59851573-5d3d-4fb7-a431-4d21e18e24d2"
+      (reference "#PWR0114") (unit 1) (value "GND") (footprint "")
+    )
+    (path "/caa71f4c-454d-4ac9-b287-456eafb34991/11143329-dd8d-4cc3-8fa4-452667b02f06"
+      (reference "#PWR0115") (unit 1) (value "GND") (footprint "")
+    )
     (path "/fc4c71a5-1008-4ac4-98db-57c838c57d91/fbc197bf-e2f3-4638-9935-f28d7c075a1e"
       (reference "CR1") (unit 1) (value "SMBJ5.0A-TR") (footprint "footprints:SMBJ5.0A-TR")
@@
       (reference "J3") (unit 1) (value "SM04B-SRSS-TB(LF)(SN)") (footprint "SM04B-SRSS-TB_LF__SN_:JST_SM04B-SRSS-TB(LF)(SN)")
     )
+    (path "/caa71f4c-454d-4ac9-b287-456eafb34991/400cdc36-083c-4c59-a2cd-106a6a90acd8"
+      (reference "J4") (unit 1) (value "USB_OTG") (footprint "CM4IO:USB_Micro-B_EDAC_UCON00686")
+    )
     (path "/fc4c71a5-1008-4ac4-98db-57c838c57d91/e653ed96-2ceb-42bc-905c-db47449cc067"
       (reference "JP1") (unit 1) (value "SolderJumper_2_Open") (footprint "Jumper:SolderJumper-2_P1.3mm_Open_RoundedPad1.0x1.5mm")
@@
     (path "/fc4c71a5-1008-4ac4-98db-57c838c57d91/463d59ed-ef45-4402-9140-190527b0aff8"
       (reference "Module1") (unit 1) (value "ComputeModule4-CM4") (footprint "CM4IO:Raspberry-Pi-4-Compute-Module")
+    )
+    (path "/caa71f4c-454d-4ac9-b287-456eafb34991/fafda8be-1326-444e-bcc1-8cb4aded3240"
+      (reference "Module1") (unit 2) (value "ComputeModule4-CM4") (footprint "CM4IO:Raspberry-Pi-4-Compute-Module")
     )
     (path "/fc4c71a5-1008-4ac4-98db-57c838c57d91/19ae9b22-a1d3-4ec4-a43e-6fb99c903f21"
@@
       (reference "R6") (unit 1) (value "1k") (footprint "Resistor_SMD:R_0603_1608Metric_Pad0.98x0.95mm_HandSolder")
     )
-    (path "/fc4c71a5-1008-4ac4-98db-57c838c57d91/862be61d-8399-4948-a564-2f01d5cb5b7a"
-      (reference "U1") (unit 1) (value "74LVC1G07SE-7") (footprint "Package_TO_SOT_SMD:SOT-353_SC-70-5")
-    )
-    (path "/caa71f4c-454d-4ac9-b287-456eafb34991/0d0caf91-4ece-48ed-a178-43a8b49f3526"
-      (reference "#PWR0111") (unit 1) (value "GND") (footprint "")
-    )
-    (path "/caa71f4c-454d-4ac9-b287-456eafb34991/81f0d702-912e-410d-83f3-c9f3bd3f7f28"
-      (reference "#PWR0112") (unit 1) (value "GND") (footprint "")
-    )
-    (path "/caa71f4c-454d-4ac9-b287-456eafb34991/7aaeccae-7554-4237-a159-f19729377488"
-      (reference "#PWR0113") (unit 1) (value "GND") (footprint "")
-    )
-    (path "/caa71f4c-454d-4ac9-b287-456eafb34991/59851573-5d3d-4fb7-a431-4d21e18e24d2"
-      (reference "#PWR0114") (unit 1) (value "GND") (footprint "")
-    )
-    (path "/caa71f4c-454d-4ac9-b287-456eafb34991/11143329-dd8d-4cc3-8fa4-452667b02f06"
-      (reference "#PWR0115") (unit 1) (value "GND") (footprint "")
-    )
-    (path "/caa71f4c-454d-4ac9-b287-456eafb34991/400cdc36-083c-4c59-a2cd-106a6a90acd8"
-      (reference "J4") (unit 1) (value "USB_OTG") (footprint "CM4IO:USB_Micro-B_EDAC_UCON00686")
-    )
-    (path "/caa71f4c-454d-4ac9-b287-456eafb34991/fafda8be-1326-444e-bcc1-8cb4aded3240"
-      (reference "Module1") (unit 2) (value "ComputeModule4-CM4") (footprint "CM4IO:Raspberry-Pi-4-Compute-Module")
-    )
     (path "/caa71f4c-454d-4ac9-b287-456eafb34991/f98e44b3-cc4b-4d36-9b5b-fc739b8abd51"
       (reference "R7") (unit 1) (value "2.2K 1%") (footprint "Resistor_SMD:R_0603_1608Metric_Pad0.98x0.95mm_HandSolder")
@@
       (reference "R8") (unit 1) (value "2.2K 1%") (footprint "Resistor_SMD:R_0603_1608Metric_Pad0.98x0.95mm_HandSolder")
     )
+    (path "/fc4c71a5-1008-4ac4-98db-57c838c57d91/862be61d-8399-4948-a564-2f01d5cb5b7a"
+      (reference "U1") (unit 1) (value "74LVC1G07SE-7") (footprint "Package_TO_SOT_SMD:SOT-353_SC-70-5")
+    )
     (path "/caa71f4c-454d-4ac9-b287-456eafb34991/25c200c8-8d48-421b-ac68-c53b8df4e956"
